File: RP2040_minimal_r2/RP2040_minimal_r2.kicad_pcb (KiCad board)
At the start: 2 copper layers, 52 x 51 mm, 34 parts, among them J1 USB_B_Micro, J2 Conn_01x02, J3 Conn_02x18_Odd_Even, J4 Conn_02x18_Odd_Even, U1 NCP1117-3.3_SOT223, U2 W25Q128JVS, U3 RP2040, Y1 ABM8-272-T3

Commit message: started some pcb design ig
Parts:
- removed C17: 10u, Capacitor_SMD:C_0805_2012Metric
- removed H1, H2, H3, H4: MountingHole, MountingHole:MountingHole_2.7mm_M2.5
- removed J1: USB_B_Micro, RP2040_minimal:USB_Micro-B_Amphenol_10103594-0001LF_Horizontal_modified
- removed J2: Conn_01x02, Connector_PinHeader_2.54mm:PinHeader_1x02_P2.54mm_Vertical
- removed J3, J4: Conn_02x18_Odd_Even, Connector_PinHeader_2.54mm:PinHeader_2x18_P2.54mm_Vertical
- added C18: 1u, Capacitor_SMD:C_0805_2012Metric, F.Cu at (150.0, 127.0)
- added C19: 4.7u, Capacitor_SMD:C_0805_2012Metric, F.Cu at (150.5, 140.5)
- added C20: 470p, Capacitor_SMD:C_0805_2012Metric, F.Cu at (153.7, 75.2)
- added C21: 0.1u, Capacitor_SMD:C_0805_2012Metric, F.Cu at (236.0, 112.0)
- added C22: 0.1u, Capacitor_SMD:C_0805_2012Metric, F.Cu at (236.0, 115.5)
- added C23: 0.1u, Capacitor_SMD:C_0805_2012Metric, F.Cu at (236.0, 108.5)
- added C24: 1u, Capacitor_SMD:C_0805_2012Metric, F.Cu at (159.5, 124.5)
- added C25: 1u, Capacitor_SMD:C_0805_2012Metric, F.Cu at (154.5, 124.5)
- added C26: 1u, Capacitor_SMD:C_0805_2012Metric, F.Cu at (159.5, 128.0)
- added C27: 1u, Capacitor_SMD:C_0805_2012Metric, F.Cu at (159.5, 131.5)
- added C28: 1u, Capacitor_SMD:C_0805_2012Metric, F.Cu at (159.5, 135.0)
- added C29: 10u, Capacitor_SMD:C_0805_2012Metric, F.Cu at (144.0, 141.0)
- added D2: 1N4148WS, Diode_SMD:D_SOD-323, F.Cu at (135.5, 137.0)
- added D3: 1N5822, Diode_THT:D_DO-201AD_P15.24mm_Horizontal, F.Cu at (153.9, 91.6)
- added D4: 1N5822, Diode_THT:D_DO-201AD_P15.24mm_Horizontal, F.Cu at (245.0, 32.0)
- added J5: Conn_01x05_Pin, Connector_JST:JST_EH_S5B-EH_1x05_P2.50mm_Horizontal, F.Cu at (175.5, 121.0)
- added J6: Conn_01x02_Pin, Connector_AMASS:AMASS_XT30PW-F_1x02_P2.50mm_Horizontal, F.Cu at (252.5, 99.7)
- added J7: Conn_01x02_Pin, Connector_AMASS:AMASS_XT30PW-F_1x02_P2.50mm_Horizontal, F.Cu at (226.5, 88.5)
- added P1: USB_C_Plug_USB2.0, Connector_USB:USB_C_Receptacle_GCT_USB4105-xx-A_16P_TopMnt_Horizontal, B.Cu at (259.9, 45.7)
- added Q1: TSM340N06CP_ROG, power_nmos:TRANS_TSM340N06CP_ROG, F.Cu at (255.5, 110.0)
- added R10: 5m, Resistor_SMD:R_0805_2012Metric_Pad1.20x1.40mm_HandSolder, F.Cu at (242.0, 112.0)
- added R11: 100, Resistor_SMD:R_0805_2012Metric_Pad1.20x1.40mm_HandSolder, F.Cu at (239.0, 110.0)
- added R12: 100, Resistor_SMD:R_0805_2012Metric_Pad1.20x1.40mm_HandSolder, F.Cu at (239.0, 114.0)
- added R13: 100, Resistor_SMD:R_0805_2012Metric_Pad1.20x1.40mm_HandSolder, F.Cu at (164.5, 116.0)
- added R14: 100, Resistor_SMD:R_0805_2012Metric_Pad1.20x1.40mm_HandSolder, F.Cu at (164.5, 121.0)
- added R15: 100, Resistor_SMD:R_0805_2012Metric_Pad1.20x1.40mm_HandSolder, F.Cu at (164.5, 126.0)
- added R16: 100, Resistor_SMD:R_0805_2012Metric_Pad1.20x1.40mm_HandSolder, F.Cu at (164.5, 131.0)
- added R17: 100, Resistor_SMD:R_0805_2012Metric_Pad1.20x1.40mm_HandSolder, F.Cu at (164.5, 136.0)
- added R18: 100, Resistor_SMD:R_0805_2012Metric_Pad1.20x1.40mm_HandSolder, F.Cu at (144.0, 137.0)
- added R19: 1M, Resistor_SMD:R_0805_2012Metric_Pad1.20x1.40mm_HandSolder, F.Cu at (247.0, 110.0)
- added R20: 5.1k, Resistor_SMD:R_0805_2012Metric_Pad1.20x1.40mm_HandSolder, F.Cu at (260.5, 52.5)
- added R6: 4.7k, Resistor_SMD:R_0805_2012Metric, F.Cu at (167.0, 69.1)
- added R7: 4.7k, Resistor_SMD:R_0805_2012Metric, F.Cu at (136.5, 68.5)
- added R8: 510k, Resistor_SMD:R_0805_2012Metric, F.Cu at (182.5, 84.5)
- added R9: 10k, Resistor_SMD:R_0805_2012Metric, F.Cu at (135.5, 133.5)
- added SW1: SW_Push, Button_Switch_SMD:SW_Push_SPST_NO_Alps_SKRK, F.Cu at (223.1, 43.0)
- added U4: BQ76920PW, Package_SO:TSSOP-20_4.4x6.5mm_P0.65mm, F.Cu at (150.5, 133.5)
- R1: footprint Resistor_SMD:R_0402_1005Metric -> Resistor_SMD:R_0805_2012Metric_Pad1.20x1.40mm_HandSolder
- U2: footprint Package_SO:SOIC-8_5.23x5.23mm_P1.27mm -> Package_SO:SOP-8_3.76x4.96mm_P1.27mm
- moved C1 135.7 mm to (239.9, 45.0)
- moved C4 135.7 mm to (241.0, 57.5)
- moved U1 135.7 mm to (240.0, 51.4)
- moved C11 134.2 mm to (223.4, 63.3)
- moved C12 134.2 mm to (236.3, 67.5)
- moved C13 134.2 mm to (223.4, 67.5)
- moved C14 134.2 mm to (230.2, 72.7)
- moved C15 134.2 mm to (236.3, 62.3)
- moved C16 134.2 mm to (236.3, 60.9)
- moved C2 134.2 mm to (228.6, 75.8)
- moved C3 134.2 mm to (231.2, 75.8)
- moved C5 134.2 mm to (226.0, 49.1)
- moved C6 134.2 mm to (228.9, 58.8)
- moved C7 134.2 mm to (231.4, 72.7)
- moved C8 134.2 mm to (232.9, 59.8)
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Connections:
- net VBUS renamed /LDO_IN
Routing:
- net /GPIO29_ADC3: track 33.2 -> 0.00 mm
- net /GPIO0: track 31.8 -> 0.00 mm
- net /GPIO28_ADC2: track 31.6 -> 0.00 mm
- net /GPIO1: track 30.2 -> 0.00 mm
- net /GPIO27_ADC1: track 29.9 -> 0.00 mm
- net /GPIO2: track 28.5 -> 0.00 mm
- net /GPIO26_ADC0: track 28.3 -> 0.00 mm
- net /GPIO3: track 26.9 -> 0.00 mm
- net /GPIO25: track 26.7 -> 0.00 mm
- net /SWCLK: track 25.9 -> 0.00 mm
- net /GPIO15: track 25.4 -> 0.00 mm
- net /GPIO4: track 25.3 -> 0.00 mm
- net /GPIO24: track 25.0 -> 0.00 mm
- net /SWD: track 24.3 -> 0.00 mm
- net /GPIO14: track 23.8 -> 0.00 mm
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- added copper zone on B.Cu, net +3V3
- added copper zone on B.Cu, net /afe/BatPos
- added copper zone on F.Cu, net /afe/BatPos
- added copper zone on B.Cu, net /afe/PackNeg
- added copper zone on F.Cu, net /afe/PackNeg
- added copper zone on B.Cu, net Net-(Q1-Pad3)
- added copper zone on F.Cu, net Net-(Q1-Pad3)
- removed copper zone on F.Cu, net /LDO_IN
Other:
- board outline removed
- board text removed: "3V3"
- board text removed: "GND"
- board text removed: "GP0"
- board text removed: "GP1"
- board text removed: "GP10"
- board text removed: "GP11"
- board text removed: "GP12"
- board text removed: "GP13"
- board text removed: "GP14"
- board text removed: "GP15"
- board text removed: "GP16"
- board text removed: "GP17"
- board text removed: "GP18"
- board text removed: "GP19"
- board text removed: "GP2"
- board text removed: "GP20"
- board text removed: "GP21"
- board text removed: "GP22"
- board text removed: "GP23"
- board text removed: "GP24"
- board text removed: "GP25"
- board text removed: "GP26"
- board text removed: "GP27"
- board text removed: "GP28"
- board text removed: "GP29"
- board text removed: "GP3"
- board text removed: "GP4"
- board text removed: "GP5"
- board text removed: "GP6"
- board text removed: "GP7"
- board text removed: "GP8"
- board text removed: "GP9"
- board text removed: "Minimal Design Example REV2"
- board text removed: "Outer Row GND"
- board text removed: "RUN"
- board text removed: "Raspberry Pi RP2040"
- board text removed: "SWCLK"
- board text removed: "SWD"
- board text removed: "USB_BOOT"
