File: RP2040_minimal_r2/afe.kicad_sch (KiCad schematic)
At the start: 31 parts, among them J5 Conn_01x05_Pin, J6 Conn_01x02_Pin, J7 Conn_01x02_Pin, Q1 TSM340N06CP_ROG, U4 BQ76920PW

Commit message: started some pcb design ig
Parts:
- added D2: 1N4148WS, Diode_SMD:D_SOD-323, symbol Diode:1N4148WS
Connections:
- net BatNeg is gone; now on net GND: J7.2 (Pin_2)
- net Vbat0 is gone; now on net GND: R13.1
- net BatPos: no longer J5.1 (Pin_1), R17.1
- net GND: now also J5.1 (Pin_1); no longer J5.5 (Pin_5)
- net VBat3: now also J5.4 (Pin_4); no longer J5.2 (Pin_2)
- net TS1: now reaches R9.1, U4.6 (TS1)
- net TS1: now also D2.1 (K)
- net VCC renamed REGOUT
- net Vbat1 renamed VBat1
- net VBat1: now also J5.2 (Pin_2); no longer J5.4 (Pin_4)
- new net BOOT: D2.2 (A)
- new net VBat4: J5.5 (Pin_5), R17.1
Other:
- moved on the sheet: J6, J7, R9
